Commit message: updated arm controls, battery, msg format, and restucture dirs

File: basestationproject/frontend/public/urdf/robot.urdf (robot description, URDF)
Before this commit: robot mo, 7 links, 6 joints
Links:
- removed link base
- removed link link1
- removed link link2
- removed link link3
- removed link link4
- removed link link5
- added link link_0, mass 5; collision mesh filename=meshes/link_0.obj; visual mesh filename=meshes/link_0.obj
- added link link_1, mass 5; collision mesh filename=meshes/link_1.obj; visual mesh filename=meshes/link_1.obj
- added link link_2, mass 5; collision mesh filename=meshes/link_2.obj; visual mesh filename=meshes/link_2.obj
- added link link_3, mass 5; collision mesh filename=meshes/link_3.obj; visual mesh filename=meshes/link_3.obj
- added link link_4, mass 5; collision mesh filename=meshes/link_4.obj; visual mesh filename=meshes/link_4.obj
- added link link_5, mass 10; collision mesh filename=meshes/fre_gripper__fixed.obj; collision mesh filename=meshes/link_5.obj
Joints:
- removed joint joint1
- removed joint joint2
- removed joint joint3
- removed joint joint4
- removed joint joint5
- removed joint world_to_base
- added joint J1: type revolute, parent link_0, child link_1, origin xyz=0.0809077 1.48087e-17 0.028 rpy=3.14159 -9.91271e-17 1.75639e-48, axis 0 0 1, limit lower=-1.5708 upper=1.5708 effort=1000 velocity=1000
- added joint J2: type revolute, parent link_1, child link_2, origin xyz=0.0855 -1.39264e-05 -0.056 rpy=-1.5708 -6.12323e-17 1.5708, axis 0 0 1, limit lower=-1.5708 upper=2.44346 effort=1000 velocity=1000
- added joint J3: type revolute, parent link_2, child link_3, origin xyz=2.76827e-16 0.45 0.0405 rpy=2.51629e-16 -8.53162e-16 -1.77023e-14, axis 0 0 1, limit lower=-1.8326 upper=2.87979 effort=1000 velocity=1000
- added joint J4: type revolute, parent link_3, child link_4, origin xyz=1.04906e-09 0.39 -0.015 rpy=-2.88523e-28 3.54659e-14 1.5708, axis 0 0 1, limit lower=-1.309 upper=2.35619 effort=1000 velocity=1000
- added joint J5: type revolute, parent link_4, child link_5, origin xyz=0.105 3.43113e-14 -0.036 rpy=1.5708 3.82745e-33 -1.5708, axis 0 0 1, limit lower=-1.5708 upper=1.5708 effort=1000 velocity=1000
- added joint world_to_link_0: type fixed, parent world, child link_0, origin xyz=0 0 0.51 rpy=0 0 0
